File: hardware/kicad/project/02_MCU_Debug_Memory.kicad_sch (KiCad schematic)
At the start: 0 parts

Commit message: feat(hardware): TB-HW-002 — populate all 12 schematic sheets with components
Populated 235 component symbols across all 12 KiCad schematic sheets:
- 01_Power: Reverse polarity, TVS (SMCJ33A), buck (LMR33630), LDO (TPS7A1633), VREF (REF5050) — 30 symbols
- 02_MCU: S32K344 (6 units), clock (40MHz+32kHz), decoupling, reset, boot config, LEDs — 30 symbols
- 03_CAN: 4x TJA1043 with CM chokes (ACT45B-510), split termination, bus filter caps — 36 symbols
- 04_USB: Molex USB-C, TPD2EUSB30 ESD, CC resistors, eFuse, Ethernet PHY footprint — 9 symbols
- 05_Inputs: 8 analog channels (RC+clamp), 2x CJ125 WBO2, 2x TLE2072 knock amps — 50 symbols
- 06_Injectors: TLE8888-2QK (8-ch P&H), flyback diodes, current sense — 14 symbols
- 07_Ignition: 6x ISL9V3040S3 IGBTs with gate resistors (100R), pull-downs (10k) — 24 symbols
- 08_Outputs: DRV8873 ETC H-bridge, TLE8110ED low-side (boost+relays), BTS4140N tach — 12 symbols
- 09_Protection: TPS3850G33 watchdog, safe-state FET, ESD diodes (PESD5V0) — 14 symbols
- 10_Connectors: 42-pin Deutsch DTM (2 units), 2x CAN 4-pin, diagnostic 4-pin — 5 symbols
- 11_Programming: TC2050 SWD, 8 test points, production security notes — 11 symbols
- 00_Cover: Block diagram, BOM summary, spec references, revision history

Symbol library: 18 custom symbols with complete pin assignments
Components from COMPONENT_SELECTION.md r0.1
42-pin connector per INTERFACE_SPECIFICATION.md (authority)
All MCU pins per MCU_SELECTION.md pin allocation
Other:
- note added: "40 MHz crystal (NX5032GA) + 32.768 kHz RTC | Guard ring required, no traces under crystal"
- note added: "BOOT_CFG[1:0] = 00 (boot from internal P-Flash)"
- note added: "Decoupling: 4x 0.1uF + 10uF + 100uF Tant per VDD_HV bank | 2x 2.2uF per V15 pin"
- note added: "Ethernet RMII (unpopulated — for V2): TI DP83848 / Microchip KSZ8081 footprint only"
- note added: "FRAM MB85RS256B (optional) — SPI bus, 256 Kb | Not populated on V1 prototype"
- note added: "MCU CORE, DEBUG & MEMORY — Sheet 02"
- note added: "NXP S32K344-EVB reference | AN13537 Hardware Design Guidelines"
- note added: "NXP S32K344EHT1VPBST | HLQFP176 EP | ARM Cortex-M7 Lockstep @ 160 MHz"
- note added: "RESET: 10k pull-up to +3V3, 100nF to GND, push-button for dev"
- note added: "Ref: docs/hardware/MCU_SELECTION.md | docs/hardware/POWER_ARCHITECTURE.md §6"
- note added: "STATUS (GREEN) + FAULT (RED) LEDs with 470R current limiting"
- note removed: "40 MHz crystal | PLL to 160 MHz | 257-QFP | External watchdog (TPS3850)"
- note removed: "MCU CORE — S32K344 | Sheet 02"
- note removed: "NXP S32K344 | 2MB Flash | 512KB SRAM | 4x CAN FD | ARM Cortex-M7 @ 160MHz"
- note removed: "Ref: docs/hardware/MCU_SELECTION.md | NXP S32K344-EVB | AN13537"

Commit message: feat(hardware): swap MCU to STM32F407VG, wire power sheet + MCU sheet
MCU CHANGE:
- Replaced NXP S32K344 with STM32F407VG (LQFP-100)
- Added STM32F407VG symbol (70 pins mapped: power, system, debug, GPIO banks)
- rusEFI firmware already targets this MCU — no firmware port needed
- Updated Sheet 01 title block, Sheet 02 fully rewritten for STM32

SCHEMATIC WIRING (Sheet 01_Power):
- GND bus rail spanning full sheet width (Y=145)
- All decoupling caps (C20-C25) connected to +3V3 rail and GND
- All bulk caps (C1-C11) connected to +5V/+3V3/+5VREF and GND
- Existing power chain hierarchy preserved (Fuse -> TVS -> FET -> Buck -> LDO -> VREF)

SCHEMATIC WIRING (Sheet 02_MCU):
- Single-unit STM32F407VG symbol placed at center
- VDD/VSS connected to +3V3/GND global labels
- VCAP pins, PDR_ON pull-up, BOOT0 pull-down wired
- 8MHz crystal + 22pF caps + bias resistor wired
- SWD header (TC2050) with pull-up resistor wired
- Crystal input/output nets connected

DESIGN PACKAGE:
- Product platform updated from S32K344 to STM32F407VG
- Firmware reference updated to f407-discovery target
Other:
- note added: "MCU CORE — Sheet 02"
- note added: "Ref: docs/hardware/MCU_SELECTION.md | COMPONENT_SELECTION.md"
- note added: "STM32F407VGT6 (LQFP-100) | 8MHz Main Crystal | 1MHz Internal RC for RTC | SWD via Tag-Connect TC2050"
- note added: "VCAP_1 (74) → 2.2uF to GND | VCAP_2 (32) → 2.2uF to GND | PDR_ON (18) → pull-up to VDD"
- note added: "VDD pins: 6, 13, 19, 72, 99 (all tied to +3V3) | VSS pins: 7, 14, 20, 73, 100 (all tied to GND)"
- note removed: "40 MHz crystal (NX5032GA) + 32.768 kHz RTC | Guard ring required, no traces under crystal"
- note removed: "BOOT_CFG[1:0] = 00 (boot from internal P-Flash)"
- note removed: "Decoupling: 4x 0.1uF + 10uF + 100uF Tant per VDD_HV bank | 2x 2.2uF per V15 pin"
- note removed: "Ethernet RMII (unpopulated — for V2): TI DP83848 / Microchip KSZ8081 footprint only"
- note removed: "FRAM MB85RS256B (optional) — SPI bus, 256 Kb | Not populated on V1 prototype"
- note removed: "MCU CORE, DEBUG & MEMORY — Sheet 02"
- note removed: "NXP S32K344-EVB reference | AN13537 Hardware Design Guidelines"
- note removed: "NXP S32K344EHT1VPBST | HLQFP176 EP | ARM Cortex-M7 Lockstep @ 160 MHz"
- note removed: "RESET: 10k pull-up to +3V3, 100nF to GND, push-button for dev"
- note removed: "Ref: docs/hardware/MCU_SELECTION.md | docs/hardware/POWER_ARCHITECTURE.md §6"
- note removed: "STATUS (GREEN) + FAULT (RED) LEDs with 470R current limiting"
- title: 7100CPT ECU — MCU Core, Debug & Memory -> 7100CPT ECU — MCU Core (STM32F407VG)
