File: hardware/kicad/project/01_Power.kicad_sch (KiCad schematic)
At the start: 0 parts

Commit message: feat(hardware): TB-HW-002 — populate all 12 schematic sheets with components
Populated 235 component symbols across all 12 KiCad schematic sheets:
- 01_Power: Reverse polarity, TVS (SMCJ33A), buck (LMR33630), LDO (TPS7A1633), VREF (REF5050) — 30 symbols
- 02_MCU: S32K344 (6 units), clock (40MHz+32kHz), decoupling, reset, boot config, LEDs — 30 symbols
- 03_CAN: 4x TJA1043 with CM chokes (ACT45B-510), split termination, bus filter caps — 36 symbols
- 04_USB: Molex USB-C, TPD2EUSB30 ESD, CC resistors, eFuse, Ethernet PHY footprint — 9 symbols
- 05_Inputs: 8 analog channels (RC+clamp), 2x CJ125 WBO2, 2x TLE2072 knock amps — 50 symbols
- 06_Injectors: TLE8888-2QK (8-ch P&H), flyback diodes, current sense — 14 symbols
- 07_Ignition: 6x ISL9V3040S3 IGBTs with gate resistors (100R), pull-downs (10k) — 24 symbols
- 08_Outputs: DRV8873 ETC H-bridge, TLE8110ED low-side (boost+relays), BTS4140N tach — 12 symbols
- 09_Protection: TPS3850G33 watchdog, safe-state FET, ESD diodes (PESD5V0) — 14 symbols
- 10_Connectors: 42-pin Deutsch DTM (2 units), 2x CAN 4-pin, diagnostic 4-pin — 5 symbols
- 11_Programming: TC2050 SWD, 8 test points, production security notes — 11 symbols
- 00_Cover: Block diagram, BOM summary, spec references, revision history

Symbol library: 18 custom symbols with complete pin assignments
Components from COMPONENT_SELECTION.md r0.1
42-pin connector per INTERFACE_SPECIFICATION.md (authority)
All MCU pins per MCU_SELECTION.md pin allocation
Other:
- note added: "6-36V -> Reverse Polarity (IPD90P04P4L) -> TVS (SMCJ33A) -> Buck (LMR33630) -> LDO (TPS7A1633) -> VREF (REF5050)"
- note added: "Decoupling: 4x 0.1uF + 2x 10uF distributed on +3V3 rail"
- note added: "F1: 30A ATO blade fuse, through-hole for field replacement"
- note added: "Power Budget: 3.3V @ 390mA max | 5V @ 55mA max | 12V @ 28A peak | Fuse: 30A ATO"
- note added: "Ref: docs/hardware/POWER_ARCHITECTURE.md | COMPONENT_SELECTION.md rows P1-P10"
- note removed: "6-36V input -> Reverse Polarity -> TVS -> Buck (12V->5V) -> LDO (5V->3.3V) -> VREF (5.0V)"
- note removed: "Key parts: IPD90P04P4L-04 (rev pol), SMCJ33A (TVS), LMR33630 (buck), TPS3850 (watchdog)"
- note removed: "Ref: docs/hardware/POWER_ARCHITECTURE.md | REUSE_MATRIX.md rows P1-P10"

Commit message: feat(hardware): swap MCU to STM32F407VG, wire power sheet + MCU sheet
MCU CHANGE:
- Replaced NXP S32K344 with STM32F407VG (LQFP-100)
- Added STM32F407VG symbol (70 pins mapped: power, system, debug, GPIO banks)
- rusEFI firmware already targets this MCU — no firmware port needed
- Updated Sheet 01 title block, Sheet 02 fully rewritten for STM32

SCHEMATIC WIRING (Sheet 01_Power):
- GND bus rail spanning full sheet width (Y=145)
- All decoupling caps (C20-C25) connected to +3V3 rail and GND
- All bulk caps (C1-C11) connected to +5V/+3V3/+5VREF and GND
- Existing power chain hierarchy preserved (Fuse -> TVS -> FET -> Buck -> LDO -> VREF)

SCHEMATIC WIRING (Sheet 02_MCU):
- Single-unit STM32F407VG symbol placed at center
- VDD/VSS connected to +3V3/GND global labels
- VCAP pins, PDR_ON pull-up, BOOT0 pull-down wired
- 8MHz crystal + 22pF caps + bias resistor wired
- SWD header (TC2050) with pull-up resistor wired
- Crystal input/output nets connected

DESIGN PACKAGE:
- Product platform updated from S32K344 to STM32F407VG
- Firmware reference updated to f407-discovery target
Changed lines of the file:
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@@
   (wire (pts (xy 150 180) (xy 150 200)) (stroke (width 0) (type default)))
   (wire (pts (xy 50 150) (xy 200 150)) (stroke (width 0) (type default)))
-  (wire (pts (xy 200 150) (xy 200 150)) (stroke (width 0) (type default)))
   (wire (pts (xy 200 190) (xy 200 150)) (stroke (width 0) (type default)))
   (wire (pts (xy 230 210) (xy 250 210)) (stroke (width 0) (type default)))
@@
   (wire (pts (xy 420 210) (xy 530 210)) (stroke (width 0) (type default)))
   (wire (pts (xy 530 210) (xy 550 210)) (stroke (width 0) (type default)))
+  (wire (pts (xy 50 145) (xy 50 100)) (stroke (width 0) (type default)) (uuid gnd_bus_01))
+  (wire (pts (xy 50 145) (xy 580 145)) (stroke (width 0) (type default)) (uuid gnd_bus_02))
+  (wire (pts (xy 170 226) (xy 170 210)) (stroke (width 0) (type default)) (uuid c1_5v_01))
+  (wire (pts (xy 170 241) (xy 170 245) (xy 580 245) (xy 580 145)) (stroke (width 0) (type default)) (uuid c1_gnd_01))
+  (wire (pts (xy 200 200) (xy 200 210)) (stroke (width 0) (type default)) (uuid buck_vout_01))
+  (wire (pts (xy 150 226) (xy 150 210)) (stroke (width 0) (type default)) (uuid c3_5v_01))
+  (wire (pts (xy 150 220) (xy 150 145)) (stroke (width 0) (type default)) (uuid c3_gnd_01))
+  (wire (pts (xy 230 226) (xy 230 210)) (stroke (width 0) (type default)) (uuid c4_5v_01))
+  (wire (pts (xy 230 241) (xy 230 145)) (stroke (width 0) (type default)) (uuid c4_gnd_01))
+  (wire (pts (xy 250 226) (xy 250 210)) (stroke (width 0) (type default)) (uuid c6_5v_01))
+  (wire (pts (xy 250 220) (xy 250 145)) (stroke (width 0) (type default)) (uuid c6_gnd_01))
+  (wire (pts (xy 360 226) (xy 360 210)) (stroke (width 0) (type default)) (uuid c7_3v3_01))
+  (wire (pts (xy 360 241) (xy 360 145)) (stroke (width 0) (type default)) (uuid c7_gnd_01))
+  (wire (pts (xy 400 226) (xy 400 210)) (stroke (width 0) (type default)) (uuid c8_3v3_01))
+  (wire (pts (xy 400 220) (xy 400 145)) (stroke (width 0) (type default)) (uuid c8_gnd_01))
+  (wire (pts (xy 415 226) (xy 415 210)) (stroke (width 0) (type default)) (uuid c9_3v3_01))
+  (wire (pts (xy 415 241) (xy 415 145)) (stroke (width 0) (type default)) (uuid c9_gnd_01))
+  (wire (pts (xy 405 241) (xy 405 145)) (stroke (width 0) (type default)) (uuid fb1_gnd_01))
+  (wire (pts (xy 530 226) (xy 530 210)) (stroke (width 0) (type default)) (uuid c10_3v3_02))
+  (wire (pts (xy 530 241) (xy 530 145)) (stroke (width 0) (type default)) (uuid c10_gnd_01))
+  (wire (pts (xy 570 226) (xy 570 210)) (stroke (width 0) (type default)) (uuid c11_5vref_01))
+  (wire (pts (xy 570 241) (xy 570 145)) (stroke (width 0) (type default)) (uuid c11_gnd_01))
+  (wire (pts (xy 200 86) (xy 200 65) (xy 50 65) (xy 50 100)) (stroke (width 0) (type default)) (uuid c20_gnd_01))
+  (wire (pts (xy 240 86) (xy 240 65) (xy 50 65) (xy 50 100)) (stroke (width 0) (type default)) (uuid c21_gnd_01))
+  (wire (pts (xy 280 86) (xy 280 65) (xy 50 65) (xy 50 100)) (stroke (width 0) (type default)) (uuid c22_gnd_01))
+  (wire (pts (xy 320 86) (xy 320 65) (xy 50 65) (xy 50 100)) (stroke (width 0) (type default)) (uuid c23_gnd_01))
+  (wire (pts (xy 360 86) (xy 360 65) (xy 50 65) (xy 50 100)) (stroke (width 0) (type default)) (uuid c24_gnd_01))
+  (wire (pts (xy 400 86) (xy 400 65) (xy 50 65) (xy 50 100)) (stroke (width 0) (type default)) (uuid c25_gnd_01))
+  (wire (pts (xy 200 80) (xy 200 65) (xy 50 65)) (stroke (width 0) (type default)) (uuid decap_3v3_01))
+  (wire (pts (xy 240 80) (xy 240 65)) (stroke (width 0) (type default)) (uuid decap_3v3_02))
+  (wire (pts (xy 280 80) (xy 280 65)) (stroke (width 0) (type default)) (uuid decap_3v3_03))
+  (wire (pts (xy 320 80) (xy 320 65)) (stroke (width 0) (type default)) (uuid decap_3v3_04))
+  (wire (pts (xy 360 80) (xy 360 65)) (stroke (width 0) (type default)) (uuid decap_3v3_05))
+  (wire (pts (xy 400 80) (xy 400 65)) (stroke (width 0) (type default)) (uuid decap_3v3_06))
+  (wire (pts (xy 50 65) (xy 50 80)) (stroke (width 0) (type default)) (uuid decap_3v3_bus))
+  (label "+3V3" (at 50 65 0) (effects (font (size 1.27 1.27))) (uuid label_3v3_decap))
+  (label "GND" (at 580 145 2) (effects (font (size 1.27 1.27))) (uuid label_gnd_end))
   (sheet_instances
     (path "/01_power/" (page "2"))
