File: hardware/kicad/project/03_CAN.kicad_sch (KiCad schematic)
At the start: 0 parts

Commit message: feat(hardware): TB-HW-002 — populate all 12 schematic sheets with components
Populated 235 component symbols across all 12 KiCad schematic sheets:
- 01_Power: Reverse polarity, TVS (SMCJ33A), buck (LMR33630), LDO (TPS7A1633), VREF (REF5050) — 30 symbols
- 02_MCU: S32K344 (6 units), clock (40MHz+32kHz), decoupling, reset, boot config, LEDs — 30 symbols
- 03_CAN: 4x TJA1043 with CM chokes (ACT45B-510), split termination, bus filter caps — 36 symbols
- 04_USB: Molex USB-C, TPD2EUSB30 ESD, CC resistors, eFuse, Ethernet PHY footprint — 9 symbols
- 05_Inputs: 8 analog channels (RC+clamp), 2x CJ125 WBO2, 2x TLE2072 knock amps — 50 symbols
- 06_Injectors: TLE8888-2QK (8-ch P&H), flyback diodes, current sense — 14 symbols
- 07_Ignition: 6x ISL9V3040S3 IGBTs with gate resistors (100R), pull-downs (10k) — 24 symbols
- 08_Outputs: DRV8873 ETC H-bridge, TLE8110ED low-side (boost+relays), BTS4140N tach — 12 symbols
- 09_Protection: TPS3850G33 watchdog, safe-state FET, ESD diodes (PESD5V0) — 14 symbols
- 10_Connectors: 42-pin Deutsch DTM (2 units), 2x CAN 4-pin, diagnostic 4-pin — 5 symbols
- 11_Programming: TC2050 SWD, 8 test points, production security notes — 11 symbols
- 00_Cover: Block diagram, BOM summary, spec references, revision history

Symbol library: 18 custom symbols with complete pin assignments
Components from COMPONENT_SELECTION.md r0.1
42-pin connector per INTERFACE_SPECIFICATION.md (authority)
All MCU pins per MCU_SELECTION.md pin allocation
Other:
- note added: "4x TJA1043TK/1Y | CAN FD 5 Mbps | Split Termination (60R+60R+4.7nF) | CM Choke ACT45B-510"
- note added: "CAN0 (Powertrain)"
- note added: "CAN1 (Body/Chassis)"
- note added: "CAN2 (Diagnostic)"
- note added: "CAN3 (Spare/Expansion)"
- note added: "EMC: CM choke ACT45B-510 on all 4 channels | Split term | Bus filter 100pF to GND | Ferrite bead on VCC"
- note added: "Ref: docs/hardware/CAN_DESIGN.md | COMPONENT_SELECTION.md rows C1-C8"
- note added: "Termination: NOT on PCB. External 120R at diag tool end."
- note added: "Unpopulated by default. Pads only."
- note removed: "4x CAN FD channels | TJA1043GT/3 transceivers | 5 Mbps FD data rate"
- note removed: "CM choke (ACT45B-510-2P-TL003) per channel | Split termination (60+60 Ohm +4.7nF)"
- note removed: "Ref: docs/hardware/CAN_DESIGN.md | REUSE_MATRIX.md rows C1-C4"
