File: hardware/kicad/project/05_Inputs_WBO2.kicad_sch (KiCad schematic)
At the start: 0 parts

Commit message: feat(hardware): TB-HW-002 — populate all 12 schematic sheets with components
Populated 235 component symbols across all 12 KiCad schematic sheets:
- 01_Power: Reverse polarity, TVS (SMCJ33A), buck (LMR33630), LDO (TPS7A1633), VREF (REF5050) — 30 symbols
- 02_MCU: S32K344 (6 units), clock (40MHz+32kHz), decoupling, reset, boot config, LEDs — 30 symbols
- 03_CAN: 4x TJA1043 with CM chokes (ACT45B-510), split termination, bus filter caps — 36 symbols
- 04_USB: Molex USB-C, TPD2EUSB30 ESD, CC resistors, eFuse, Ethernet PHY footprint — 9 symbols
- 05_Inputs: 8 analog channels (RC+clamp), 2x CJ125 WBO2, 2x TLE2072 knock amps — 50 symbols
- 06_Injectors: TLE8888-2QK (8-ch P&H), flyback diodes, current sense — 14 symbols
- 07_Ignition: 6x ISL9V3040S3 IGBTs with gate resistors (100R), pull-downs (10k) — 24 symbols
- 08_Outputs: DRV8873 ETC H-bridge, TLE8110ED low-side (boost+relays), BTS4140N tach — 12 symbols
- 09_Protection: TPS3850G33 watchdog, safe-state FET, ESD diodes (PESD5V0) — 14 symbols
- 10_Connectors: 42-pin Deutsch DTM (2 units), 2x CAN 4-pin, diagnostic 4-pin — 5 symbols
- 11_Programming: TC2050 SWD, 8 test points, production security notes — 11 symbols
- 00_Cover: Block diagram, BOM summary, spec references, revision history

Symbol library: 18 custom symbols with complete pin assignments
Components from COMPONENT_SELECTION.md r0.1
42-pin connector per INTERFACE_SPECIFICATION.md (authority)
All MCU pins per MCU_SELECTION.md pin allocation
Other:
- note added: "12 Analog Channels: TPS(x2), MAP, CLT, IAT, WBO2(x2), KNOCK(x2), FP, OP, VBAT"
- note added: "CLT: NTC thermistor, 2.49k bias to VREF"
- note added: "FP: 0-5V, ratiometric"
- note added: "IAT: NTC thermistor, 2.49k bias to VREF"
- note added: "KNOCK SENSOR AMPLIFIERS"
- note added: "Knock #1: TLE2072 bandpass filter, biased VREF/2"
- note added: "Knock #2: TLE2072 bandpass filter, biased VREF/2"
- note added: "MAP: 0-5V, ratiometric"
- note added: "OP: 0-5V, ratiometric"
- note added: "Ref: docs/hardware/PROTECTION_CIRCUITS.md §4, §6 | COMPONENT_SELECTION.md rows I1-I10"
- note added: "TPS1: 0-5V, ratiometric, 10k pull-down"
- note added: "TPS2: Safety redundant, 10k pull-down"
- note added: "VBAT_SENSE: 1:10 divider from VBAT, R38+R39"
- note added: "WBO2 #1: CJ125 + IRLR2905 heater driver | 0.1R current sense"
- note added: "WBO2 #2: CJ125 + IRLR2905 heater driver | 0.1R current sense"
- note added: "WIDEBAND O2 SENSORS"
- note removed: "BAV99 clamp diodes on all external inputs | 5.0V VREF from REF5050"
- note removed: "RC filtered analog inputs (1k + 10nF) | WBO2 via CJ125 | Knock sensor conditioning"
- note removed: "Ref: docs/hardware/INTERFACE_SPECIFICATION.md | REUSE_MATRIX.md rows I1-I12"
