File: hardware/kicad/project/09_Protection.kicad_sch (KiCad schematic)
At the start: 0 parts

Commit message: feat(hardware): TB-HW-002 — populate all 12 schematic sheets with components
Populated 235 component symbols across all 12 KiCad schematic sheets:
- 01_Power: Reverse polarity, TVS (SMCJ33A), buck (LMR33630), LDO (TPS7A1633), VREF (REF5050) — 30 symbols
- 02_MCU: S32K344 (6 units), clock (40MHz+32kHz), decoupling, reset, boot config, LEDs — 30 symbols
- 03_CAN: 4x TJA1043 with CM chokes (ACT45B-510), split termination, bus filter caps — 36 symbols
- 04_USB: Molex USB-C, TPD2EUSB30 ESD, CC resistors, eFuse, Ethernet PHY footprint — 9 symbols
- 05_Inputs: 8 analog channels (RC+clamp), 2x CJ125 WBO2, 2x TLE2072 knock amps — 50 symbols
- 06_Injectors: TLE8888-2QK (8-ch P&H), flyback diodes, current sense — 14 symbols
- 07_Ignition: 6x ISL9V3040S3 IGBTs with gate resistors (100R), pull-downs (10k) — 24 symbols
- 08_Outputs: DRV8873 ETC H-bridge, TLE8110ED low-side (boost+relays), BTS4140N tach — 12 symbols
- 09_Protection: TPS3850G33 watchdog, safe-state FET, ESD diodes (PESD5V0) — 14 symbols
- 10_Connectors: 42-pin Deutsch DTM (2 units), 2x CAN 4-pin, diagnostic 4-pin — 5 symbols
- 11_Programming: TC2050 SWD, 8 test points, production security notes — 11 symbols
- 00_Cover: Block diagram, BOM summary, spec references, revision history

Symbol library: 18 custom symbols with complete pin assignments
Components from COMPONENT_SELECTION.md r0.1
42-pin connector per INTERFACE_SPECIFICATION.md (authority)
All MCU pins per MCU_SELECTION.md pin allocation
Other:
- note added: "CONNECTOR ESD PROTECTION"
- note added: "EXTERNAL WATCHDOG"
- note added: "External Watchdog (TPS3850) | Safe-State FET | ESD Diodes | 30A Fuse"
- note added: "PESD5V0 ESD diodes on all external-facing connector pins (analog, digital inputs)"
- note added: "PROTECTION — Sheet 09"
- note added: "Ref: docs/hardware/PROTECTION_CIRCUITS.md | COMPONENT_SELECTION.md rows P1-P8"
- note added: "SAFE-STATE CUTOFF"
- note added: "Safe-state P-MOSFET: cuts VBAT to injectors, ignition, ETC on watchdog timeout"
- note added: "TPS3850G33: Window watchdog, 1.6-2.6s window | 49.9k C_SET resistor"
- note added: "WDI from MCU GPIO (toggle every ~2s) | ~WDO -> Safe-State FET gate | ~RST -> MCU ~RESET"
- note removed: "30A input fuse | ESD on all connectors | TVS on all external pins"
- note removed: "External watchdog: TPS3850 (200ms timeout) | Safe-state FET cuts 12V output rail"
- note removed: "PROTECTION & SAFETY — Sheet 09"
- note removed: "Ref: docs/hardware/PROTECTION_CIRCUITS.md | REUSE_MATRIX.md rows S1-S8"
Changed lines of the file:
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@@
-(kicad_sch (version 20240108) (generator "eeschema")
+(kicad_sch (version 20240108) (generator "7100CPT-schematic-gen")
   (paper "A3")
   (title_block
     (title "7100CPT ECU — Watchdog, Safe State, ESD")
     (date "2026-07-03")
-    (rev "0.1")
+    (rev "0.2")
     (company "${COMPANY}")
-    (comment 1 "External watchdog (TPS3850), safe-state FET, ESD, fuses (30A)")
+    (comment 1 "TPS3850 watchdog, safe-state FET, ESD diodes, 30A fuse")
     (comment 2 "NXP S32K344 | rusEFI Firmware | IPC Class 3")
     (comment 3 "High-Tg FR-4 (TG170+) | ENIG | 1.6 mm")
-    (comment 4 "REUSE_MATRIX.md — NXP Reference Following")
+    (comment 4 "Phase 0 Approved | REUSE_MATRIX gate passed")
     (comment 5 "-40C to +85C | IP67 Target | 6-Layer")
   )
-  (symbol_instances)
-  (text "PROTECTION & SAFETY — Sheet 09"
-    (at 25 24 0) (effects (font (size 3.0 3.0) bold) (justify left bottom)))
-  (text "External watchdog: TPS3850 (200ms timeout) | Safe-state FET cuts 12V output rail"
-    (at 25 30 0) (effects (font (size 1.5 1.5)) (justify left bottom)))
-  (text "30A input fuse | ESD on all connectors | TVS on all external pins"
-    (at 25 36 0) (effects (font (size 1.5 1.5)) (justify left bottom)))
-  (text "Ref: docs/hardware/PROTECTION_CIRCUITS.md | REUSE_MATRIX.md rows S1-S8"
-    (at 25 42 0) (effects (font (size 1.27 1.27)) (justify left bottom)))
+  (symbol_instances
+  (symbol (lib_id "7100CPT:TPS3850G33") (at 150 200 0) (unit 1)
+    (exclude_from_sim yes) (in_bom yes) (on_board yes) (dnp no)
+    (property "Reference" "U45" (at 150 200 0) (effects (font (size 1.27 1.27))))
+    (property "Value" "TPS3850G33DRCR" (at 150 193.65 0) (effects (font (size 1.27 1.27))))
+  )
+  (symbol (lib_id "Device:R") (at 110 200 0) (unit 1)
+    (exclude_from_sim yes) (in_bom yes) (on_board yes) (dnp no)
+    (property "Reference" "R110" (at 110 200 0) (effects (font (size 1.27 1.27))))
+    (property "Value" "49.9k" (at 110 193.65 0) (effects (font (size 1.27 1.27))))
+  )
+  (symbol (lib_id "Device:R") (at 110 185 0) (unit 1)
+    (exclude_from_sim yes) (in_bom yes) (on_board yes) (dnp no)
+    (property "Reference" "R111" (at 110 185 0) (effects (font (size 1.27 1.27))))
+    (property "Value" "100k" (at 110 178.65 0) (effects (font (size 1.27 1.27))))
+  )
+  (symbol (lib_id "Device:R") (at 190 185 0) (unit 1)
+    (exclude_from_sim yes) (in_bom yes) (on_board yes) (dnp no)
+    (property "Reference" "R112" (at 190 185 0) (effects (font (size 1.27 1.27))))
+    (property "Value" "100k" (at 190 178.65 0) (effects (font (size 1.27 1.27))))
+  )
+  (symbol (lib_id "7100CPT:IPD90P04P4L") (at 180 140 0) (unit 1)
+    (exclude_from_sim yes) (in_bom yes) (on_board yes) (dnp no)
+    (property "Reference" "Q30" (at 180 140 0) (effects (font (size 1.27 1.27))))
+    (property "Value" "IPD90P04P4L-04" (at 180 133.65 0) (effects (font (size 1.27 1.27))))
+  )
+  (symbol (lib_id "Device:R") (at 180 125 0) (unit 1)
+    (exclude_from_sim yes) (in_bom yes) (on_board yes) (dnp no)
+    (property "Reference" "R113" (at 180 125 0) (effects (font (size 1.27 1.27))))
+    (property "Value" "100k" (at 180 118.65 0) (effects (font (size 1.27 1.27))))
+  )
+  (symbol (lib_id "Device:D_TVS") (at 50 100 0) (unit 1)
+    (exclude_from_sim yes) (in_bom yes) (on_board yes) (dnp no)
+    (property "Reference" "D60" (at 50 100 0) (effects (font (size 1.27 1.27))))
+    (property "Value" "PESD5V0" (at 50 93.65 0) (effects (font (size 1.27 1.27))))
+  )
+  (symbol (lib_id "Device:D_TVS") (at 120 100 0) (unit 1)
+    (exclude_from_sim yes) (in_bom yes) (on_board yes) (dnp no)
+    (property "Reference" "D61" (at 120 100 0) (effects (font (size 1.27 1.27))))
+    (property "Value" "PESD5V0" (at 120 93.65 0) (effects (font (size 1.27 1.27))))
+  )
+  (symbol (lib_id "Device:D_TVS") (at 190 100 0) (unit 1)
+    (exclude_from_sim yes) (in_bom yes) (on_board yes) (dnp no)
+    (property "Reference" "D62" (at 190 100 0) (effects (font (size 1.27 1.27))))
+    (property "Value" "PESD5V0" (at 190 93.65 0) (effects (font (size 1.27 1.27))))
+  )
+  (symbol (lib_id "Device:D_TVS") (at 260 100 0) (unit 1)
+    (exclude_from_sim yes) (in_bom yes) (on_board yes) (dnp no)
+    (property "Reference" "D63" (at 260 100 0) (effects (font (size 1.27 1.27))))
+    (property "Value" "PESD5V0" (at 260 93.65 0) (effects (font (size 1.27 1.27))))
+  )
+  (symbol (lib_id "Device:D_TVS") (at 330 100 0) (unit 1)
+    (exclude_from_sim yes) (in_bom yes) (on_board yes) (dnp no)
+    (property "Reference" "D64" (at 330 100 0) (effects (font (size 1.27 1.27))))
+    (property "Value" "PESD5V0" (at 330 93.65 0) (effects (font (size 1.27 1.27))))
+  )
+  (symbol (lib_id "Device:D_TVS") (at 400 100 0) (unit 1)
+    (exclude_from_sim yes) (in_bom yes) (on_board yes) (dnp no)
+    (property "Reference" "D65" (at 400 100 0) (effects (font (size 1.27 1.27))))
+    (property "Value" "PESD5V0" (at 400 93.65 0) (effects (font (size 1.27 1.27))))
+  )
+  (symbol (lib_id "Device:D_TVS") (at 470 100 0) (unit 1)
+    (exclude_from_sim yes) (in_bom yes) (on_board yes) (dnp no)
+    (property "Reference" "D66" (at 470 100 0) (effects (font (size 1.27 1.27))))
+    (property "Value" "PESD5V0" (at 470 93.65 0) (effects (font (size 1.27 1.27))))
+  )
+  (symbol (lib_id "Device:D_TVS") (at 540 100 0) (unit 1)
+    (exclude_from_sim yes) (in_bom yes) (on_board yes) (dnp no)
+    (property "Reference" "D67" (at 540 100 0) (effects (font (size 1.27 1.27))))
+    (property "Value" "PESD5V0" (at 540 93.65 0) (effects (font (size 1.27 1.27))))
+  )
+  )
+  (text "PROTECTION — Sheet 09" (at 25 250 0) (effects (font (size 3.0 3.0) bold) (justify left bottom)))
+  (text "External Watchdog (TPS3850) | Safe-State FET | ESD Diodes | 30A Fuse" (at 25 244 0) (effects (font (size 1.5 1.5)) (justify left bottom)))
+  (text "EXTERNAL WATCHDOG" (at 25 220 0) (effects (font (size 1.5 1.5) bold) (justify left bottom)))
+  (text "TPS3850G33: Window watchdog, 1.6-2.6s window | 49.9k C_SET resistor" (at 25 180 0) (effects (font (size 1.27 1.27)) (justify left bottom)))
+  (text "WDI from MCU GPIO (toggle every ~2s) | ~WDO -> Safe-State FET gate | ~RST -> MCU ~RESET" (at 25 173 0) (effects (font (size 1.27 1.27)) (justify left bottom)))
+  (text "SAFE-STATE CUTOFF" (at 25 160 0) (effects (font (size 1.5 1.5) bold) (justify left bottom)))
+  (text "Safe-state P-MOSFET: cuts VBAT to injectors, ignition, ETC on watchdog timeout" (at 25 115 0) (effects (font (size 1.27 1.27)) (justify left bottom)))
+  (text "CONNECTOR ESD PROTECTION" (at 25 115 0) (effects (font (size 1.5 1.5) bold) (justify left bottom)))
+  (text "PESD5V0 ESD diodes on all external-facing connector pins (analog, digital inputs)" (at 25 85 0) (effects (font (size 1.27 1.27)) (justify left bottom)))
+  (text "Ref: docs/hardware/PROTECTION_CIRCUITS.md | COMPONENT_SELECTION.md rows P1-P8" (at 25 70 0) (effects (font (size 1.27 1.27)) (justify left bottom)))
+  (global_label "+3V3" (shape input) (at 150 210 0) (effects (font (size 1.27 1.27))))
+  (global_label "GND" (shape input) (at 150 190 0) (effects (font (size 1.27 1.27))))
+  (global_label "GND" (shape input) (at 110 185 0) (effects (font (size 1.27 1.27))))
+  (global_label "GND" (shape input) (at 190 185 0) (effects (font (size 1.27 1.27))))
+  (global_label "VBAT" (shape input) (at 180 150 0) (effects (font (size 1.27 1.27))))
+  (global_label "VBAT_PROTECTED" (shape input) (at 200 140 0) (effects (font (size 1.27 1.27))))
+  (global_label "GND" (shape input) (at 180 120 0) (effects (font (size 1.27 1.27))))
+  (global_label "GND" (shape input) (at 50 90 0) (effects (font (size 1.27 1.27))))
+  (global_label "GND" (shape input) (at 120 90 0) (effects (font (size 1.27 1.27))))
+  (global_label "GND" (shape input) (at 190 90 0) (effects (font (size 1.27 1.27))))
+  (global_label "GND" (shape input) (at 260 90 0) (effects (font (size 1.27 1.27))))
+  (global_label "GND" (shape input) (at 330 90 0) (effects (font (size 1.27 1.27))))
+  (global_label "GND" (shape input) (at 400 90 0) (effects (font (size 1.27 1.27))))
+  (global_label "GND" (shape input) (at 470 90 0) (effects (font (size 1.27 1.27))))
+  (global_label "GND" (shape input) (at 540 90 0) (effects (font (size 1.27 1.27))))
   (sheet_instances
     (path "/09_protection/" (page "10"))
