File: hardware/kicad/project/10_Connectors.kicad_sch (KiCad schematic)
At the start: 0 parts

Commit message: fix(hardware): ship prep — connector migration, library paths, MCU refs, Sheet 11 wiring
🔴 Connector: 42-pin Deutsch DTM → 35-pin AMPSEAL 16
  - Created AMPSEAL16_35PIN + DTM04_4PIN (WBO2) symbols in library
  - Rewrote Sheet 10 with AMPSEAL connector + WBO2 pigtail connectors
  - Updated INTERFACE_SPECIFICATION.md with full 35-pin pinout
  - Signal consolidation: dropped KNOCK2, OP, RELAY_SP; WBO2→dedicated Deutsch

🔴 Library path: sym-lib-table + fp-lib-table now point to ../ dirs
  (fixes KiCad not finding custom symbols/footprints)

🔴 MCU refs: All 11 sheets + root ECU.kicad_sch + cover ASCII art
  updated from NXP S32K344 → STM32F407VG

🟡 Sheet 11: Added global labels (+3V3, SWDIO, SWCLK, SWO, ~RESET, +5V)
  and wired TC2050 debug header through series resistors to signal nets

📄 Docs: DESIGN_PACKAGE.md, DESIGN_NOTES.md, INTERFACE_SPECIFICATION.md
  all updated to reflect current state
Other:
- note added: "34 active signals + 1 NC | Gold-plated socket cavities | 14-22 AWG per pin function"
- note added: "35-Pin AMPSEAL 16 Main Harness | CAN x2 (4-pin Deutsch) | WBO2 x2 (4-pin Deutsch) | Diag (4-pin Deutsch)"
- note added: "CAN BUS CONNECTORS (2x 4-Pin Deutsch DTM)"
- note added: "CAN0 (Powertrain): Pin1=GND, Pin2=CAN0_H, Pin3=CAN0_L, Pin4=VBAT(fused)"
- note added: "CAN1 (Body/Exp): Pin1=GND, Pin2=CAN1_H, Pin3=CAN1_L, Pin4=VBAT(fused)"
- note added: "CAN2_Diag: Pin1=GND, Pin2=CAN2_H, Pin3=CAN2_L, Pin4=VBAT(1A fused)"
- note added: "MAIN HARNESS CONNECTOR — 35-Pin AMPSEAL 16 (TE 1-967648-1)"
- note added: "Pin1=GND, Pin2=LAMBDA, Pin3=HEATER, Pin4=VBAT — 4-wire LSU 4.9 wideband"
- note added: "Pins 1-2: Power | 3-11: Injectors | 12-20: Ignition | 21-22: ETC | 23-27: Sensors | 28-34: Outputs/Relays/Spare"
- note added: "Ref: docs/hardware/INTERFACE_SPECIFICATION.md | TE AMPSEAL 16 series | Deutsch DTM series"
- note added: "WBO2 SENSOR CONNECTORS (2x 4-Pin Deutsch DTM)"
- note removed: "34-Pin AMPSEAL 16 | CAN x2 (4-pin Deutsch) | Diag (4-pin Deutsch) | USB-C | SWD | Expansion"
- note removed: "CAN CONNECTORS (2x 4-Pin Deutsch DTM)"
- note removed: "CAN0: Pin1=GND, Pin2=CAN_H, Pin3=CAN_L, Pin4=VBAT(fused)"
- note removed: "CAN1: Pin1=GND, Pin2=CAN_H, Pin3=CAN_L, Pin4=VBAT(fused)"
- note removed: "CAN2 diagnostic port: Pin1=GND, Pin2=CAN2_H, Pin3=CAN2_L, Pin4=VBAT(1A fused)"
- note removed: "MAIN HARNESS CONNECTOR — 34-Pin AMPSEAL 16"
- note removed: "Mating: AMPSEAL 16 plug | Gold-plated sockets | 14-22 AWG per pin function"
- note removed: "Pin Summary: Main 34-pin (30 used, 4 spare) | CAN x2 (8 used) | Diag (4 used) | USB-C (4 used) | DEBUG (5 used)"
- note removed: "Pins 1-17: Power, Injectors, Ignition | Pins 18-34: ETC, Sensors, WBO2, Knock, Boost, Relays"
- note removed: "Ref: docs/hardware/INTERFACE_SPECIFICATION.md §1-6 | TE Connectivity AMPSEAL 16 series"
- note removed: "USB-C: Molex 105450-0101 — see Sheet 04_USB"
- title: 7100CPT ECU — 34-Pin AMPSEAL, CAN, USB, SWD, Expansion -> 7100CPT ECU — 35-Pin AMPSEAL, CAN, USB, SWD, Expansion
Changed lines of the file:
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@@
   (paper "A3")
   (title_block
-    (title "7100CPT ECU — 34-Pin AMPSEAL, CAN, USB, SWD, Expansion")
-    (date "2026-07-03")
-    (rev "0.2")
+    (title "7100CPT ECU — 35-Pin AMPSEAL, CAN, USB, SWD, Expansion")
+    (date "2026-07-11")
+    (rev "0.3")
     (company "${COMPANY}")
-    (comment 1 "Main harness (34-pin AMPSEAL 16), CAN x2, diagnostic port, USB-C, debug")
-    (comment 2 "NXP S32K344 | rusEFI Firmware | IPC Class 3")
+    (comment 1 "Main harness (35-pin AMPSEAL 16), CAN x2, WBO2 x2, diag port, USB-C, debug")
+    (comment 2 "STM32F407VG | rusEFI Firmware | IPC Class 3")
     (comment 3 "High-Tg FR-4 (TG170+) | ENIG | 1.6 mm")
-    (comment 4 "Phase 0 Approved | REUSE_MATRIX gate passed")
+    (comment 4 "TB-HW-003 — Connector sheet wired, AMPSEAL migration complete")
     (comment 5 "-40C to +85C | IP67 Target | 6-Layer")
   )
   (symbol_instances
-  (symbol (lib_id "7100CPT:DTM_42PIN") (at 100 200 0) (unit 1)
+  ;; === MAIN HARNESS — 35-Pin AMPSEAL 16 ===
+  (symbol (lib_id "7100CPT:AMPSEAL16_35PIN") (at 200 250 0) (unit 1)
     (exclude_from_sim yes) (in_bom yes) (on_board yes) (dnp no)
-    (property "Reference" "J1A" (at 100 200 0) (effects (font (size 1.27 1.27))))
-    (property "Value" "DTM06-12SA_Bank_A" (at 100 193.65 0) (effects (font (size 1.27 1.27))))
+    (property "Reference" "J1" (at 200 250 0) (effects (font (size 1.27 1.27))))
+    (property "Value" "AMPSEAL16_35POS" (at 200 243.65 0) (effects (font (size 1.27 1.27))))
   )
-  (symbol (lib_id "7100CPT:DTM_42PIN") (at 100 120 0) (unit 2)
+  ;; === CAN CONNECTORS — 4-Pin Deutsch DTM ===
+  (symbol (lib_id "Connector:Conn_01x04_Male") (at 50 200 0) (unit 1)
     (exclude_from_sim yes) (in_bom yes) (on_board yes) (dnp no)
-    (property "Reference" "J1B" (at 100 120 0) (effects (font (size 1.27 1.27))))
-    (property "Value" "DTM06-12SA_Bank_B" (at 100 113.65 0) (effects (font (size 1.27 1.27))))
+    (property "Reference" "J3" (at 50 200 0) (effects (font (size 1.27 1.27))))
+    (property "Value" "DTM06-4S_CAN0" (at 50 193.65 0) (effects (font (size 1.27 1.27))))
   )
-  (symbol (lib_id "Connector:Conn_01x04_Male") (at 50 70 0) (unit 1)
+  (symbol (lib_id "Connector:Conn_01x04_Male") (at 250 200 0) (unit 1)
     (exclude_from_sim yes) (in_bom yes) (on_board yes) (dnp no)
-    (property "Reference" "J3" (at 50 70 0) (effects (font (size 1.27 1.27))))
-    (property "Value" "DTM06-4S_CAN0" (at 50 63.65 0) (effects (font (size 1.27 1.27))))
+    (property "Reference" "J4" (at 250 200 0) (effects (font (size 1.27 1.27))))
+    (property "Value" "DTM06-4S_CAN1" (at 250 193.65 0) (effects (font (size 1.27 1.27))))
   )
-  (symbol (lib_id "Connector:Conn_01x04_Male") (at 250 70 0) (unit 1)
+  (symbol (lib_id "Connector:Conn_01x04_Male") (at 450 200 0) (unit 1)
     (exclude_from_sim yes) (in_bom yes) (on_board yes) (dnp no)
-    (property "Reference" "J4" (at 250 70 0) (effects (font (size 1.27 1.27))))
-    (property "Value" "DTM06-4S_CAN1" (at 250 63.65 0) (effects (font (size 1.27 1.27))))
+    (property "Reference" "J5" (at 450 200 0) (effects (font (size 1.27 1.27))))
+    (property "Value" "DTM06-4S_DIAG" (at 450 193.65 0) (effects (font (size 1.27 1.27))))
   )
-  (symbol (lib_id "Connector:Conn_01x04_Male") (at 50 30 0) (unit 1)
+  ;; === WBO2 CONNECTORS — 4-Pin Deutsch DTM ===
+  (symbol (lib_id "7100CPT:DTM04_4PIN") (at 50 120 0) (unit 1)
     (exclude_from_sim yes) (in_bom yes) (on_board yes) (dnp no)
-    (property "Reference" "J5" (at 50 30 0) (effects (font (size 1.27 1.27))))
-    (property "Value" "DTM06-4S_DIAG" (at 50 23.65 0) (effects (font (size 1.27 1.27))))
+    (property "Reference" "J6" (at 50 120 0) (effects (font (size 1.27 1.27))))
+    (property "Value" "DTM06-4S_WBO2_1" (at 50 113.65 0) (effects (font (size 1.27 1.27))))
+  )
+  (symbol (lib_id "7100CPT:DTM04_4PIN") (at 250 120 0) (unit 1)
+    (exclude_from_sim yes) (in_bom yes) (on_board yes) (dnp no)
+    (property "Reference" "J7" (at 250 120 0) (effects (font (size 1.27 1.27))))
+    (property "Value" "DTM06-4S_WBO2_2" (at 250 113.65 0) (effects (font (size 1.27 1.27))))
   )
   )
-  (text "CONNECTORS — Sheet 10" (at 25 260 0) (effects (font (size 3.0 3.0) bold) (justify left bottom)))
-  (text "34-Pin AMPSEAL 16 | CAN x2 (4-pin Deutsch) | Diag (4-pin Deutsch) | USB-C | SWD | Expansion" (at 25 254 0) (effects (font (size 1.5 1.5)) (justify left bottom)))
-  (text "MAIN HARNESS CONNECTOR — 34-Pin AMPSEAL 16" (at 25 230 0) (effects (font (size 1.5 1.5) bold) (justify left bottom)))
-  (text "Pins 1-17: Power, Injectors, Ignition | Pins 18-34: ETC, Sensors, WBO2, Knock, Boost, Relays" (at 100 100 0) (effects (font (size 1.27 1.27)) (justify left bottom)))
-  (text "Mating: AMPSEAL 16 plug | Gold-plated sockets | 14-22 AWG per pin function" (at 100 93 0) (effects (font (size 1.27 1.27)) (justify left bottom)))
-  (text "CAN CONNECTORS (2x 4-Pin Deutsch DTM)" (at 25 90 0) (effects (font (size 1.5 1.5) bold) (justify left bottom)))
-  (text "CAN0: Pin1=GND, Pin2=CAN_H, Pin3=CAN_L, Pin4=VBAT(fused)" (at 50 55 0) (effects (font (size 1.0 1.0)) (justify left bottom)))
-  (text "CAN1: Pin1=GND, Pin2=CAN_H, Pin3=CAN_L, Pin4=VBAT(fused)" (at 250 55 0) (effects (font (size 1.0 1.0)) (justify left bottom)))
-  (text "DIAGNOSTIC CONNECTOR (4-Pin Deutsch DTM)" (at 25 50 0) (effects (font (size 1.5 1.5) bold) (justify left bottom)))
-  (text "CAN2 diagnostic port: Pin1=GND, Pin2=CAN2_H, Pin3=CAN2_L, Pin4=VBAT(1A fused)" (at 50 15 0) (effects (font (size 1.0 1.0)) (justify left bottom)))
-  (text "USB-C: Molex 105450-0101 — see Sheet 04_USB" (at 400 50 0) (effects (font (size 1.27 1.27)) (justify left bottom)))
-  (text "Pin Summary: Main 34-pin (30 used, 4 spare) | CAN x2 (8 used) | Diag (4 used) | USB-C (4 used) | DEBUG (5 used)" (at 25 -10 0) (effects (font (size 1.27 1.27)) (justify left bottom)))
-  (text "Ref: docs/hardware/INTERFACE_SPECIFICATION.md §1-6 | TE Connectivity AMPSEAL 16 series" (at 25 -17 0) (effects (font (size 1.27 1.27)) (justify left bottom)))
+  ;; === SHEET TITLES ===
+  (text "CONNECTORS — Sheet 10" (at 25 330 0) (effects (font (size 3.0 3.0) bold) (justify left bottom)))
+  (text "35-Pin AMPSEAL 16 Main Harness | CAN x2 (4-pin Deutsch) | WBO2 x2 (4-pin Deutsch) | Diag (4-pin Deutsch)" (at 25 324 0) (effects (font (size 1.5 1.5)) (justify left bottom)))
+  (text "MAIN HARNESS CONNECTOR — 35-Pin AMPSEAL 16 (TE 1-967648-1)" (at 25 295 0) (effects (font (size 1.5 1.5) bold) (justify left bottom)))
+  (text "34 active signals + 1 NC | Gold-plated socket cavities | 14-22 AWG per pin function" (at 25 285 0) (effects (font (size 1.27 1.27)) (justify left bottom)))
+  (text "Pins 1-2: Power | 3-11: Injectors | 12-20: Ignition | 21-22: ETC | 23-27: Sensors | 28-34: Outputs/Relays/Spare" (at 25 275 0) (effects (font (size 1.27 1.27)) (justify left bottom)))
+  (text "CAN BUS CONNECTORS (2x 4-Pin Deutsch DTM)" (at 25 215 0) (effects (font (size 1.5 1.5) bold) (justify left bottom)))
+  (text "CAN0 (Powertrain): Pin1=GND, Pin2=CAN0_H, Pin3=CAN0_L, Pin4=VBAT(fused)" (at 50 185 0) (effects (font (size 1.27 1.27)) (justify left bottom)))
+  (text "CAN1 (Body/Exp):  Pin1=GND, Pin2=CAN1_H, Pin3=CAN1_L, Pin4=VBAT(fused)" (at 250 185 0) (effects (font (size 1.27 1.27)) (justify left bottom)))
+  (text "DIAGNOSTIC CONNECTOR (4-Pin Deutsch DTM)" (at 25 155 0) (effects (font (size 1.5 1.5) bold) (justify left bottom)))
+  (text "CAN2_Diag: Pin1=GND, Pin2=CAN2_H, Pin3=CAN2_L, Pin4=VBAT(1A fused)" (at 450 185 0) (effects (font (size 1.27 1.27)) (justify left bottom)))
+  (text "WBO2 SENSOR CONNECTORS (2x 4-Pin Deutsch DTM)" (at 25 130 0) (effects (font (size 1.5 1.5) bold) (justify left bottom)))
+  (text "Pin1=GND, Pin2=LAMBDA, Pin3=HEATER, Pin4=VBAT — 4-wire LSU 4.9 wideband" (at 50 105 0) (effects (font (size 1.27 1.27)) (justify left bottom)))
+  (text "Ref: docs/hardware/INTERFACE_SPECIFICATION.md | TE AMPSEAL 16 series | Deutsch DTM series" (at 25 75 0) (effects (font (size 1.27 1.27)) (justify left bottom)))
   (sheet_instances
     (path "/10_connectors/" (page "11"))
