File: hardware/kicad/project/ECU.kicad_sch (KiCad schematic)
At the start: 12 parts

Commit message: fix(hardware): ship prep — connector migration, library paths, MCU refs, Sheet 11 wiring
🔴 Connector: 42-pin Deutsch DTM → 35-pin AMPSEAL 16
  - Created AMPSEAL16_35PIN + DTM04_4PIN (WBO2) symbols in library
  - Rewrote Sheet 10 with AMPSEAL connector + WBO2 pigtail connectors
  - Updated INTERFACE_SPECIFICATION.md with full 35-pin pinout
  - Signal consolidation: dropped KNOCK2, OP, RELAY_SP; WBO2→dedicated Deutsch

🔴 Library path: sym-lib-table + fp-lib-table now point to ../ dirs
  (fixes KiCad not finding custom symbols/footprints)

🔴 MCU refs: All 11 sheets + root ECU.kicad_sch + cover ASCII art
  updated from NXP S32K344 → STM32F407VG

🟡 Sheet 11: Added global labels (+3V3, SWDIO, SWCLK, SWO, ~RESET, +5V)
  and wired TC2050 debug header through series resistors to signal nets

📄 Docs: DESIGN_PACKAGE.md, DESIGN_NOTES.md, INTERFACE_SPECIFICATION.md
  all updated to reflect current state
Other:
- note added: "STM32F407VG | 12 Hierarchical Sheets | IPC Class 3"
- note removed: "NXP S32K344 | 12 Hierarchical Sheets | IPC Class 3"
Changed lines of the file:
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@@
     (comment 1 "12 Hierarchical Sheets")
     (comment 2 "Architecture: Phase 0 Approved | REUSE_MATRIX.md gate passed")
-    (comment 3 "NXP S32K344-EVB reference | AN13537 | CISPR 25 Class 3")
+    (comment 3 "STM32F407VG-EVAL reference | AN13537 | CISPR 25 Class 3")
     (comment 4 "IPC Class 3 | High-Tg FR-4 TG170+ | ENIG | 1.6 mm")
     (comment 5 "-40C to +85C | IP67 Target | 6-Layer | 2oz Power, 1oz Signal")
@@
     (effects (font (size 3.0 3.0) bold) (justify left bottom))
   )
-  (text "NXP S32K344 | 12 Hierarchical Sheets | IPC Class 3"
+  (text "STM32F407VG | 12 Hierarchical Sheets | IPC Class 3"
     (at 25 30 0)
     (effects (font (size 2.0 2.0)) (justify left bottom))
